File: KiCAD/HubBoard/_saved_HubBoard.sch (KiCad schematic (older format))
At the start: 51 parts, among them CN1 CONN_WHITE_5, CN2 CONN_RED_2_Power, CN3 CONN_WHITE_5, SW1 SLIDE_SW, U1 DF3_UART, U10 PSOC3_CY8C38_FAMILY_100, U2 DF3_UART, U3 DF3_UART, U4 DF3_UART, U5 TA48M05F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

Commit message: update
Parts:
- added CN4: CONN_RED_2_Power, symbol CONN_RED_2_Power
- C27: footprint Capacitors_SMD:C_0603 -> Capacitors_ThroughHole:C_Radial_D5_L6_P2.5
- CP1: footprint Capacitors_ThroughHole:C_Radial_D6.3_L11.2_P2.5 -> Capacitors_ThroughHole:C_Radial_D10_L13_P5
- CP2: footprint Capacitors_ThroughHole:C_Radial_D14_L25_P5 -> Capacitors_ThroughHole:C_Radial_D10_L13_P5
Connections:
- net +24V: now also CN4.1 (+)
- net +5V: now also U8.75 (VDDIO0); no longer U1.1 (VCC), U2.1 (VCC), U3.1 (VCC), U4.1 (VCC)
- net +9V: now also U1.1 (VCC), U2.1 (VCC), U3.1 (VCC), U4.1 (VCC)
- net GND: now also U8.66 (VSSD), CN4.2 (-)
- no-connect marks 98 -> 116
