File: KiCAD/HubBoard/HubBoard_5x10.kicad_pcb (KiCad board)
At the start: 2 copper layers, 90 x 60 mm, 56 parts, among them CN1 CONN_WHITE_5, CN2 DF22L-2P, CN3 CONN_WHITE_5, CN4 DF22R-2P, CN5 CONN_WHITE_3, CN6 CONN_WHITE_3, SW1 SLIDE_SW, U1 DF3_UART, U10 PSOC3_CY8C38_FAMILY_100, U11 drill_3mm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

Commit message: new branch
Parts:
- removed CN5, CN6: CONN_WHITE_3, user_conn:DF1E-3P_Streight
- removed D2: LED, Diodes_ThroughHole:Diode_DO-41_SOD81_Vertical_AnodeUp
- removed R4: R, Resistors_ThroughHole:Resistor_Horizontal_RM10mm
- removed U11, U12, U13, U9: drill_3mm, Wire_Pads:SolderWirePad_single_1-5mmDrill
- added C1: 1u, Capacitors_SMD:C_0805, B.Cu at (109.8, 83.5)
- added C14: 1u, Capacitors_SMD:C_0805, B.Cu at (65.9, 126.5)
- added C15: 1u, Capacitors_SMD:C_0805, B.Cu at (69.2, 126.5)
- added C2: 1u, Capacitors_SMD:C_0805, B.Cu at (106.0, 83.5)
- D1: footprint Diodes_ThroughHole:Diode_DO-41_SOD81_Vertical_AnodeUp -> Diodes_ThroughHole:Diode_DO-35_SOD27_Horizontal_RM10
- U7: footprint user_conn:USB_MINI_B_HIROSE -> Capacitors_SMD:C_0603
- moved U1 68.8 mm to (244.0, 89.0)
- moved U7 66.9 mm to (248.5, 75.0), turned to 180 degrees
- moved U2 66.0 mm to (226.0, 89.0)
- moved Y2 63.2 mm to (191.0, 93.0)
- moved CN4 61.7 mm to (231.0, 56.0)
- moved C20 59.4 mm to (201.0, 98.2), turned to 270 degrees
- moved C3 59.0 mm to (119.2, 66.0), turned to 90 degrees
- moved C21 58.9 mm to (181.0, 98.2), turned to 270 degrees
- moved CN1 57.7 mm to (218.5, 60.0), turned to 0 degrees
- moved C23 56.7 mm to (179.5, 80.0)
- moved C16 56.6 mm to (202.0, 60.2)
- moved C25 56.4 mm to (179.5, 77.8)
- moved C7 56.4 mm to (221.5, 111.2)
- moved C8 56.2 mm to (225.8, 111.8)
- moved C6 55.9 mm to (228.5, 111.8)
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Connections:
- C10 pad 1: Net-(C10-Pad1) -> +5V
- C11 pad 1: VCCD1 -> +5V
- C17 pad 1: Net-(C17-Pad1) -> +5V
- C19 pad 1: VCCD2 -> +5V
- U10 pad 27: RX_2 -> TX_1
- U10 pad 28: TX_2 -> RX_1
- U10 pad 29: RX_1 -> TX_2
- U10 pad 30: TX_1 -> RX_2
- U10 pad 31: RX_4 -> TX_3
- U10 pad 32: TX_4 -> RX_3
- U10 pad 33: RX_3 -> TX_4
- U10 pad 34: TX_3 -> RX_4
- U10 pad 37: Net-(C17-Pad1) -> +5V
- U10 pad 39: VCCD2 -> +5V
- U10 pad 86: VCCD2 -> +5V
- U8 pad 1: Net-(CN5-Pad3) -> (no net)
- U8 pad 2: Net-(CN5-Pad2) -> (no net)
- U8 pad 24: Net-(CN6-Pad3) -> (no net)
- U8 pad 25: Net-(CN6-Pad2) -> (no net)
- U8 pad 35: Net-(U7-Pad3) -> (no net)
- U8 pad 37: Net-(C10-Pad1) -> +5V
- U8 pad 39: VCCD1 -> +5V
- U8 pad 86: VCCD1 -> +5V
Routing:
- net GND: track 286.0 -> 0.00 mm, vias 4 -> 0
- net +5V: track 178.9 -> 0.00 mm, vias 2 -> 0
- net +9V: track 164.7 -> 0.00 mm, vias 4 -> 0
- net Net-(CN2-Pad1): track 64.7 -> 0.00 mm
- net RX_4: track 61.8 -> 0.00 mm
- net +24V: track 58.8 -> 0.00 mm
- net TX_4: track 57.1 -> 0.00 mm
- net TX_1: track 50.8 -> 0.00 mm
- net RX_1: track 47.0 -> 0.00 mm
- net RX_3: track 44.0 -> 0.00 mm
- net TX_3: track 42.3 -> 0.00 mm
- net TX_2: track 33.5 -> 0.00 mm
- net RX_2: track 29.1 -> 0.00 mm
- net Net-(U7-Pad3): track 26.6 -> 0.00 mm, vias 2 -> 0
- net Net-(CN1-Pad2): track 24.3 -> 0.00 mm
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- removed copper zone on B.Cu, net GND
Other:
- board size 90 x 60 mm -> 100 x 50 mm
