File: KiCAD/HubBoard/HubBoard.sch (KiCad schematic (older format))
At the start: 31 parts, among them U1 PSOC3_CY8C38_FAMILY_100, Y1 Crystal

Commit message: 回路図みかん
Parts:
- gave numbers to parts that had none: 1
Changed lines of the file:
@@
 $EndComp
 $Comp
-L R R?
+L R 0.33
 U 1 1 55795307
 P 10800 5700
-F 0 "R?" V 10880 5700 50  0000 C CNN
+F 0 "0.33" V 10880 5700 50  0000 C CNN
 F 1 "R" V 10800 5700 50  0000 C CNN
 F 2 "" V 10730 5700 30  0000 C CNN

Commit message: update
Parts:
- added CN?: CONN_WHITE_5, symbol CONN_WHITE_5
- added U?: Mini-B, symbol Mini-B
Connections:
- net +5V: now also CN?.5 (P5)
- net GND: now also CN?.4 (P4), U?.5 (GND)
- net RX_4: now also U1.22 (P1[2]); no longer U1.20 (P1[0],SWDIO,TMS)
- net TX_4: now also U1.23 (P1[3],SWV,TDO); no longer U1.21 (P1[1],SWDCK,TCK)
- net at U1.15 (XRES): now also CN?.3 (P3)
- net at U1.35 (USB_D+,P15[6]): now also U?.3 (D+)
- net at U1.36 (USB_D-,P15[7]): now also U?.2 (D-)
- new net: CN?.1 (P1), U1.20 (P1[0],SWDIO,TMS)
- new net: CN?.2 (P2), U1.21 (P1[1],SWDCK,TCK)
Other:
- moved on the sheet: 0.33, 100u, 1k, 220u, 470p, 470u, 6.2k, D?, U?

Commit message: update
Parts:
- added C14, C15, C19, C23: 1u, Capacitors_SMD:C_0805, symbol C-RESCUE-HubBoard
- added C16, C17, C18, C22, C24, C25, C29: 0.1u, Capacitors_SMD:C_0603, symbol C-RESCUE-HubBoard
- added C20, C21: 12p, Capacitors_SMD:C_0603, symbol C-RESCUE-HubBoard
- added CN2: CONN_RED_2_Power, user_conn:CONN_RED_2P, symbol CONN_RED_2_Power
- added CN3: CONN_WHITE_5, user_conn:DF1E-5P_Streight, symbol CONN_WHITE_5
- added SW1: SLIDE_SW, user_SW:Toggle_Switch_2L, symbol SLIDE_SW
- added U10: PSOC3_CY8C38_FAMILY_100, Housings_QFP:TQFP-100_14x14mm_Pitch0.5mm, symbol PSOC3_CY8C38_FAMILY_100
- added Y2: Crystal, Crystals:Crystal_HC49-SD_SMD, symbol Crystal
- C1: renamed from 1u1; value C -> 1u; footprint (none) -> Capacitors_SMD:C_0805; symbol C -> C-RESCUE-HubBoard
- C10: renamed from 0.1u3; value C -> 0.1u; footprint (none) -> Capacitors_SMD:C_0603; symbol C -> C-RESCUE-HubBoard
- C11: renamed from 1u2; value C -> 1u; footprint (none) -> Capacitors_SMD:C_0805; symbol C -> C-RESCUE-HubBoard
- C12: renamed from 15p1; value C -> 12p; footprint (none) -> Capacitors_SMD:C_0603; symbol C -> C-RESCUE-HubBoard
- C13: renamed from 15p2; value C -> 12p; footprint (none) -> Capacitors_SMD:C_0603; symbol C -> C-RESCUE-HubBoard
- C2: renamed from 1u4; value C -> 1u; footprint (none) -> Capacitors_SMD:C_0805; symbol C -> C-RESCUE-HubBoard
- C26: renamed from 0.1u; value C -> 0.1u; footprint (none) -> Capacitors_SMD:C_0603; symbol C -> C-RESCUE-HubBoard
- C27: renamed from 33u; value C -> 33u; footprint (none) -> Capacitors_ThroughHole:C_Radial_D5_L6_P2.5; symbol C -> C-RESCUE-HubBoard
- C28: renamed from 0.1u2; value C -> 0.1u; footprint (none) -> Capacitors_SMD:C_0603; symbol C -> C-RESCUE-HubBoard
- C3: renamed from 0.1u1; value C -> 0.1u; footprint (none) -> Capacitors_SMD:C_0603; symbol C -> C-RESCUE-HubBoard
- C4: renamed from 0.1u4; value C -> 0.1u; footprint (none) -> Capacitors_SMD:C_0603; symbol C -> C-RESCUE-HubBoard
- C5: renamed from 0.1u5; value C -> 0.1u; footprint (none) -> Capacitors_SMD:C_0603; symbol C -> C-RESCUE-HubBoard
- C6: renamed from 1u3; value C -> 1u; footprint (none) -> Capacitors_SMD:C_0805; symbol C -> C-RESCUE-HubBoard
- C7: renamed from 0.1u6; value C -> 0.1u; footprint (none) -> Capacitors_SMD:C_0603; symbol C -> C-RESCUE-HubBoard
- C8: renamed from 0.1u7; value C -> 0.1u; footprint (none) -> Capacitors_SMD:C_0603; symbol C -> C-RESCUE-HubBoard
- C9: renamed from 470p; value C -> 470p; footprint (none) -> Capacitors_ThroughHole:C_Disc_D6_P5; symbol C -> C-RESCUE-HubBoard
- CN1: renamed from CN?; footprint (none) -> user_conn:DF1E-5P_Streight
- CP1: renamed from 470u; value CP1 -> 470u; footprint (none) -> Capacitors_ThroughHole:C_Radial_D10_L13_P5; symbol CP1 -> CP1-RESCUE-HubBoard
- CP2: renamed from 100u; value CP1 -> 100u; footprint (none) -> Capacitors_ThroughHole:C_Radial_D10_L13_P5; symbol CP1 -> CP1-RESCUE-HubBoard
- D1: renamed from D?; footprint (none) -> Diodes_ThroughHole:Diode_DO-35_SOD27_Horizontal_RM10
- L1: renamed from 220u; value INDUCTOR -> 220u; footprint (none) -> Capacitors_ThroughHole:C_Radial_D6.3_L11.2_P2.5
- R1: renamed from 1k; value R -> 1k; footprint (none) -> Resistors_ThroughHole:Resistor_Horizontal_RM10mm; symbol R -> R-RESCUE-HubBoard
- R2: renamed from 6.2k; value R -> 6.2k; footprint (none) -> Resistors_ThroughHole:Resistor_Horizontal_RM10mm; symbol R -> R-RESCUE-HubBoard
- R3: renamed from 0.33; value R -> 0.33; footprint (none) -> Resistors_ThroughHole:Resistor_Horizontal_RM10mm; symbol R -> R-RESCUE-HubBoard
- U1, U2, U3, U4: renamed from U?; footprint (none) -> user_conn:DF1E-4P
- U5: renamed from U?; footprint (none) -> user_IC:TO-251
- U6: renamed from U?; footprint (none) -> Power_Integrations:PDIP-8
- U7: renamed from U?; footprint (none) -> Capacitors_SMD:C_0603
- U8: renamed from U1; footprint (none) -> Housings_QFP:TQFP-100_14x14mm_Pitch0.5mm
- Y1: footprint (none) -> Crystals:Crystal_HC49-SD_SMD
Connections:
- net +24V: now also SW1.6
- net +5V: now also C27.1, C14.1, C15.1, C16.1, C18.1, C22.1, C24.1, C25.1, C29.1, CN3.5 (P5), U10.100 (VDDIO2), U10.26 (VDDIO1), U10.50 (VDDIO3), U10.65 (VDDA), U10.75 (VDDIO0), U10.86 (VCCD), U10.88 (VDDD); no longer U1.1 (VCC), U2.1 (VCC), U3.1 (VCC), U4.1 (VCC), U8.75 (VDDIO0)
- net +9V: now also C26.1, U1.1 (VCC), U2.1 (VCC), U3.1 (VCC), U4.1 (VCC)
- net GND: now also C12.2, C13.2, C14.2, C15.2, C16.2, C17.2, C18.2, C19.2, C20.2, C21.2, C22.2, C23.2, C24.2, C25.2, C29.2, CN2.2 (-), CN3.4 (P4), U10.10 (VSSB), U10.13 (VBAT), U10.14 (VSSD), U10.38 (VSSD), U10.64 (VSSA), U10.66 (VSSD), U10.87 (VSSD); no longer U8.66 (VSSD)
- net RX_1: now also U10.28 (P1[7]); no longer U8.1 (P2[5])
- net RX_2: now also U10.30 (P12[7],SIO); no longer U8.6 (P6[4])
- net RX_3: now also U10.32 (P5[5]); no longer U8.16 (P5[0])
- net RX_4: now also U10.34 (P5[7]); no longer U8.22 (P1[2])
- net TX_1: now also U10.27 (P1[6]); no longer U8.2 (P2[6])
- net TX_2: now also U10.29 (P12[6],SIO); no longer U8.7 (P6[5])
- net TX_3: now also U10.31 (P5[4]); no longer U8.17 (P5[1])
- net TX_4: now also U10.33 (P5[6]); no longer U8.23 (P1[3],SWV,TDO)
- net bus9: now reaches U8.89 (P6[0])
- net bus9: now also U10.98 (P2[3])
- net bus8: now reaches U8.90 (P6[1])
- net bus8: now also U10.97 (P2[2])
- net bus7: now reaches U8.91 (P6[2])
- net bus7: now also U10.96 (P2[1])
- net bus6: now reaches U8.92 (P6[3])
- net bus6: now also U10.95 (P2[0])
- net bus5: now reaches U8.93 (P15[4])
- net bus5: now also U10.94 (P15[5])
- net bus4: now reaches U8.94 (P15[5])
- net bus4: now also U10.93 (P15[4])
- net bus3: now reaches U8.95 (P2[0])
- net bus3: now also U10.92 (P6[3])
- net bus2: now reaches U8.96 (P2[1])
- net bus2: now also U10.91 (P6[2])
- net bus1: now reaches U8.97 (P2[2])
- net bus1: now also U10.90 (P6[1])
- net bus0: now reaches U8.98 (P2[3])
- net bus0: now also U10.89 (P6[0])
- new net: CN3.3 (P3), U10.15 (XRES)
- new net: CN3.1 (P1), U10.20 (P1[0],SWDIO,TMS)
- new net: CN3.2 (P2), U10.21 (P1[1],SWDCK,TCK)
- new net: C17.1, U10.37 (VDDD)
- new net: C19.1, U10.39 (VCCD)
- new net: C20.1, U10.42 (P15[0],MHZXOUT), Y2.2
- new net: C21.1, U10.43 (P15[1],MHZXIN), Y2.1
- new net: C23.1, U10.63 (VCCA)
- new net: CN2.1 (+), SW1.4, SW1.5
- no-connect marks 0 -> 98
Other:
- moved on the sheet: C1, C12, C13, C2, C26, C27, C28, C4, C5, C6, C7, C8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

Commit message: new branch
Parts:
- removed C1, C14, C15, C2: 1u, Capacitors_SMD:C_0805, symbol C-RESCUE-HubBoard
- removed CN2: CONN_RED_2_Power, user_conn:CONN_RED_2P, symbol CONN_RED_2_Power
- added CN2: DF22L-2P, user_conn:CONN_RED_2P, symbol DF22L-2P
- added CN4: DF22R-2P, user_conn:CONN_RED_2P, symbol DF22R-2P
- added CN5, CN6: CONN_WHITE_3, user_conn:DF1E-3P_Streight, symbol CONN_WHITE_3
- added D2: LED, Diodes_ThroughHole:Diode_DO-41_SOD81_Vertical_AnodeUp, symbol LED
- added R4: R, Resistors_ThroughHole:Resistor_Horizontal_RM10mm, symbol R
- added U11, U12, U13, U9: drill_3mm, Wire_Pads:SolderWirePad_single_1-5mmDrill, symbol drill_3mm
- D1: footprint Diodes_ThroughHole:Diode_DO-35_SOD27_Horizontal_RM10 -> Diodes_ThroughHole:Diode_DO-41_SOD81_Vertical_AnodeUp
- L1: footprint Capacitors_ThroughHole:C_Radial_D6.3_L11.2_P2.5 -> Resistors_ThroughHole:Resistor_Horizontal_RM10mm
- U7: footprint Capacitors_SMD:C_0603 -> user_conn:USB_MINI_B_HIROSE
Connections:
- net labels added: VCCD1, VCCD2
- wire segments 210 -> 227
- no-connect marks 98 -> 112
Other:
- moved on the sheet: C10, C11, C17, SW1

Commit message: update
Parts:
- added L2: 470u, Capacitors_ThroughHole:C_Radial_D10_L20_P7.5, symbol INDUCTOR
- D2: footprint Diodes_ThroughHole:Diode_DO-41_SOD81_Vertical_AnodeUp -> LEDs:LED-3MM
- L1: value 220u -> 470u; footprint Resistors_ThroughHole:Resistor_Horizontal_RM10mm -> Capacitors_ThroughHole:C_Radial_D10_L20_P7.5
- R4: footprint Resistors_ThroughHole:Resistor_Horizontal_RM10mm -> Resistors_SMD:R_0603
- U1, U2, U3, U4: footprint user_conn:DF1E-4P -> user_conn:DF1E-4P_Streight
Connections:
- wire segments 227 -> 231
Changed lines of the file:
@@
 F 0 "U1" H 1200 5250 60  0000 C CNN
 F 1 "DF3_UART" H 950 5800 60  0000 C CNN
-F 2 "user_conn:DF1E-4P" H 900 5500 60  0001 C CNN
+F 2 "user_conn:DF1E-4P_Streight" H 900 5500 60  0001 C CNN
 F 3 "" H 900 5500 60  0000 C CNN
 	1    950  5500
@@
 F 0 "U2" H 1200 5850 60  0000 C CNN
 F 1 "DF3_UART" H 950 6400 60  0000 C CNN
-F 2 "user_conn:DF1E-4P" H 900 6100 60  0001 C CNN
+F 2 "user_conn:DF1E-4P_Streight" H 900 6100 60  0001 C CNN
 F 3 "" H 900 6100 60  0000 C CNN
 	1    950  6100
@@
 F 0 "U3" H 1200 6450 60  0000 C CNN
 F 1 "DF3_UART" H 950 7000 60  0000 C CNN
-F 2 "user_conn:DF1E-4P" H 900 6700 60  0001 C CNN
+F 2 "user_conn:DF1E-4P_Streight" H 900 6700 60  0001 C CNN
 F 3 "" H 900 6700 60  0000 C CNN
 	1    950  6700
@@
 F 0 "U4" H 1200 7050 60  0000 C CNN
 F 1 "DF3_UART" H 950 7600 60  0000 C CNN
-F 2 "user_conn:DF1E-4P" H 900 7300 60  0001 C CNN
+F 2 "user_conn:DF1E-4P_Streight" H 900 7300 60  0001 C CNN
 F 3 "" H 900 7300 60  0000 C CNN
 	1    950  7300
@@
 P 1650 8400
 F 0 "L1" V 1600 8400 50  0000 C CNN
-F 1 "220u" V 1750 8400 50  0000 C CNN
-F 2 "Resistors_ThroughHole:Resistor_Horizontal_RM10mm" H 1650 8400 60  0001 C CNN
+F 1 "470u" V 1750 8400 50  0000 C CNN
+F 2 "Capacitors_ThroughHole:C_Radial_D10_L20_P7.5" H 1650 8400 60  0001 C CNN
 F 3 "" H 1650 8400 60  0000 C CNN
 	1    1650 8400
@@
 F 0 "D2" H 4000 8450 50  0000 C CNN
 F 1 "LED" H 4000 8250 50  0000 C CNN
-F 2 "Diodes_ThroughHole:Diode_DO-41_SOD81_Vertical_AnodeUp" H 4000 8350 60  0001 C CNN
+F 2 "LEDs:LED-3MM" H 4000 8350 60  0001 C CNN
 F 3 "" H 4000 8350 60  0000 C CNN
 	1    4000 8350
@@
 F 0 "R4" V 4080 8700 50  0000 C CNN
 F 1 "R" V 4000 8700 50  0000 C CNN
-F 2 "Resistors_ThroughHole:Resistor_Horizontal_RM10mm" V 3930 8700 30  0001 C CNN
+F 2 "Resistors_SMD:R_0603" V 3930 8700 30  0001 C CNN
 F 3 "" H 4000 8700 30  0000 C CNN
 	1    4000 8700
@@
 NoConn ~ 10600 2550
 NoConn ~ 10600 2650
+$Comp
+L INDUCTOR L2
+U 1 1 55B1EC0F
+P 1650 8150
+F 0 "L2" V 1600 8150 50  0000 C CNN
+F 1 "470u" V 1750 8150 50  0000 C CNN
+F 2 "Capacitors_ThroughHole:C_Radial_D10_L20_P7.5" H 1650 8150 60  0001 C CNN
+F 3 "" H 1650 8150 60  0000 C CNN
+	1    1650 8150
+	0    -1   -1   0
+$EndComp
+Wire Wire Line
+	1300 8400 1300 8150
+Wire Wire Line
+	1300 8150 1350 8150
+Connection ~ 1300 8400
+Wire Wire Line
+	1950 8150 2000 8150
+Wire Wire Line
+	2000 8150 2000 8400
+Connection ~ 2000 8400
 $EndSCHEMATC

Commit message: 5x10半分完成
Parts:
- removed L2: 470u, Capacitors_ThroughHole:C_Radial_D10_L20_P7.5, symbol INDUCTOR
- added D10, D7, D8, D9: LED, LEDs:LED-0603, symbol LED
- added R10, R11, R12, R9: 1k, Resistors_SMD:R_0603, symbol R
- L1: value 470u -> 220u; footprint Capacitors_ThroughHole:C_Radial_D10_L20_P7.5 -> Capacitors_ThroughHole:C_Radial_D10_L20_P5
- SW1: footprint user_SW:Toggle_Switch_2L -> user_SW:Toggle_Swith
Connections:
- wire segments 231 -> 240
- no-connect marks 112 -> 102
Changed lines of the file:
@@
 P 1650 8400
 F 0 "L1" V 1600 8400 50  0000 C CNN
-F 1 "470u" V 1750 8400 50  0000 C CNN
-F 2 "Capacitors_ThroughHole:C_Radial_D10_L20_P7.5" H 1650 8400 60  0001 C CNN
+F 1 "220u" V 1750 8400 50  0000 C CNN
+F 2 "Capacitors_ThroughHole:C_Radial_D10_L20_P5" H 1650 8400 60  0001 C CNN
 F 3 "" H 1650 8400 60  0000 C CNN
 	1    1650 8400
@@
 F 3 "" H 4300 9550 60  0000 C CNN
 	1    4300 9550
-	1    0    0    -1
-$EndComp
-$Comp
-L SLIDE_SW SW1
-U 1 1 55A3429A
-P 4650 9750
-F 0 "SW1" H 5050 9600 60  0000 C CNN
-F 1 "SLIDE_SW" H 5100 9700 60  0000 C CNN
-F 2 "user_SW:Toggle_Switch_2L" H 4650 9750 60  0001 C CNN
-F 3 "" H 4650 9750 60  0000 C CNN
-	1    4650 9750
 	1    0    0    -1
 $EndComp
@@
 NoConn ~ 6900 5550
 NoConn ~ 7000 5550
-NoConn ~ 7700 4950
-NoConn ~ 7700 4850
 NoConn ~ 7700 4750
 NoConn ~ 7700 4650
@@
 	8050 3650 8050 4200
 Connection ~ 8050 4150
+NoConn ~ 4750 9950
+NoConn ~ 4650 9950
 NoConn ~ 4550 9950
-NoConn ~ 4650 9950
-NoConn ~ 4750 9950
 Wire Wire Line
 	1200 8350 1200 8400
 Connection ~ 1200 8400
-NoConn ~ 10600 2750
-NoConn ~ 10600 2850
-NoConn ~ 10600 2950
-NoConn ~ 10600 3250
 NoConn ~ 10600 3350
 NoConn ~ 10600 3550
@@
 Wire Wire Line
 	7850 2750 8250 2750
-NoConn ~ 10600 3050
-NoConn ~ 10600 3150
 NoConn ~ 10600 4050
 NoConn ~ 10600 4150
@@
 L CONN_WHITE_3 CN5
 U 1 1 55B153A6
-P 3500 2650
-F 0 "CN5" H 3550 2900 60  0000 C CNN
-F 1 "CONN_WHITE_3" H 3550 2400 60  0000 C CNN
-F 2 "user_conn:DF1E-3P_Streight" H 3500 2650 60  0001 C CNN
-F 3 "" H 3500 2650 60  0000 C CNN
-	1    3500 2650
+P 3500 4950
+F 0 "CN5" H 3550 5200 60  0000 C CNN
+F 1 "CONN_WHITE_3" H 3550 4700 60  0000 C CNN
+F 2 "user_conn:DF1E-3P_Streight" H 3500 4950 60  0001 C CNN
+F 3 "" H 3500 4950 60  0000 C CNN
+	1    3500 4950
 	-1   0    0    1
 $EndComp
@@
 L CONN_WHITE_3 CN6
 U 1 1 55B15A77
-P 3600 4950
-F 0 "CN6" H 3650 5200 60  0000 C CNN
-F 1 "CONN_WHITE_3" H 3650 4700 60  0000 C CNN
-F 2 "user_conn:DF1E-3P_Streight" H 3600 4950 60  0001 C CNN
-F 3 "" H 3600 4950 60  0000 C CNN
-	1    3600 4950
-	-1   0    0    1
-$EndComp
-Wire Wire Line
-	3750 2550 4100 2550
-Wire Wire Line
-	4100 2650 3750 2650
+P 8200 4850
+F 0 "CN6" H 8250 5100 60  0000 C CNN
+F 1 "CONN_WHITE_3" H 8250 4600 60  0000 C CNN
+F 2 "user_conn:DF1E-3P_Streight" H 8200 4850 60  0001 C CNN
+F 3 "" H 8200 4850 60  0000 C CNN
+	1    8200 4850
+	1    0    0    -1
+$EndComp
+Wire Wire Line
+	3750 4850 4100 4850
+Wire Wire Line
+	4100 4950 3750 4950
 $Comp
 L GND #PWR062
 U 1 1 55B16535
-P 3750 2850
-F 0 "#PWR062" H 3750 2600 50  0001 C CNN
-F 1 "GND" H 3750 2700 50  0000 C CNN
-F 2 "" H 3750 2850 60  0000 C CNN
-F 3 "" H 3750 2850 60  0000 C CNN
-	1    3750 2850
-	1    0    0    -1
-$EndComp
-Wire Wire Line
-	3750 2750 3750 2850
-Wire Wire Line
-	3850 4850 4100 4850
-Wire Wire Line
-	3850 4950 4100 4950
+P 3750 5150
+F 0 "#PWR062" H 3750 4900 50  0001 C CNN
+F 1 "GND" H 3750 5000 50  0000 C CNN
+F 2 "" H 3750 5150 60  0000 C CNN
+F 3 "" H 3750 5150 60  0000 C CNN
+	1    3750 5150
+	1    0    0    -1
+$EndComp
+Wire Wire Line
+	3750 5050 3750 5150
 $Comp
 L GND #PWR063
 U 1 1 55B173F9
-P 3850 5150
-F 0 "#PWR063" H 3850 4900 50  0001 C CNN
-F 1 "GND" H 3850 5000 50  0000 C CNN
-F 2 "" H 3850 5150 60  0000 C CNN
-F 3 "" H 3850 5150 60  0000 C CNN
-	1    3850 5150
-	1    0    0    -1
-$EndComp
-Wire Wire Line
-	3850 5050 3850 5150
+P 7950 4650
+F 0 "#PWR063" H 7950 4400 50  0001 C CNN
+F 1 "GND" H 7950 4500 50  0000 C CNN
+F 2 "" H 7950 4650 60  0000 C CNN
+F 3 "" H 7950 4650 60  0000 C CNN
+	1    7950 4650
+	-1   0    0    1
+$EndComp
+Wire Wire Line
+	7950 4750 7950 4650
 NoConn ~ 10600 4950
 NoConn ~ 10600 4850
-NoConn ~ 10600 2550
-NoConn ~ 10600 2650
-$Comp
-L INDUCTOR L2
-U 1 1 55B1EC0F
-P 1650 8150
-F 0 "L2" V 1600 8150 50  0000 C CNN
-F 1 "470u" V 1750 8150 50  0000 C CNN
-F 2 "Capacitors_ThroughHole:C_Radial_D10_L20_P7.5" H 1650 8150 60  0001 C CNN
-F 3 "" H 1650 8150 60  0000 C CNN
-	1    1650 8150
+$Comp
+L SLIDE_SW SW1
+U 1 1 55A3429A
+P 4650 9750
+F 0 "SW1" H 5050 9600 60  0000 C CNN
+F 1 "SLIDE_SW" H 5100 9700 60  0000 C CNN
+F 2 "user_SW:Toggle_Swith" H 4650 9750 60  0001 C CNN
+F 3 "" H 4650 9750 60  0000 C CNN
+	1    4650 9750
+	-1   0    0    1
+$EndComp
+Wire Wire Line
+	7950 4950 7700 4950
+Wire Wire Line
+	7950 4850 7700 4850
+$Comp
+L LED D9
+U 1 1 55B4A6EA
+P 10350 3150
+F 0 "D9" H 10350 3250 50  0000 C CNN
+F 1 "LED" H 10350 3050 50  0000 C CNN
+F 2 "LEDs:LED-0603" H 10350 3150 60  0001 C CNN
+F 3 "" H 10350 3150 60  0000 C CNN
+	1    10350 3150
+	1    0    0    -1
+$EndComp
+$Comp
+L LED D8
+U 1 1 55B4A77F
+P 10350 3050
+F 0 "D8" H 10350 3150 50  0000 C CNN
+F 1 "LED" H 10350 2950 50  0000 C CNN
+F 2 "LEDs:LED-0603" H 10350 3050 60  0001 C CNN
+F 3 "" H 10350 3050 60  0000 C CNN
+	1    10350 3050
+	1    0    0    -1
+$EndComp
+$Comp
+L LED D7
+U 1 1 55B4A81A
+P 10350 2950
+F 0 "D7" H 10350 3050 50  0000 C CNN
+F 1 "LED" H 10350 2850 50  0000 C CNN
+F 2 "LEDs:LED-0603" H 10350 2950 60  0001 C CNN
+F 3 "" H 10350 2950 60  0000 C CNN
+	1    10350 2950
+	1    0    0    -1
+$EndComp
+$Comp
+L LED D10
+U 1 1 55B4A8C1
+P 10350 3250
+F 0 "D10" H 10350 3350 50  0000 C CNN
+F 1 "LED" H 10350 3150 50  0000 C CNN
+F 2 "LEDs:LED-0603" H 10350 3250 60  0001 C CNN
+F 3 "" H 10350 3250 60  0000 C CNN
+	1    10350 3250
+	1    0    0    -1
+$EndComp
+Wire Wire Line
+	10550 2950 10600 2950
+Wire Wire Line
+	10550 3050 10600 3050
+Wire Wire Line
+	10550 3150 10600 3150
+Wire Wire Line
+	10550 3250 10600 3250
+$Comp
+L R R9
+U 1 1 55B4E3E4
+P 9950 2950
+F 0 "R9" V 10030 2950 50  0000 C CNN
+F 1 "1k" V 9950 2950 50  0000 C CNN
+F 2 "Resistors_SMD:R_0603" V 9880 2950 30  0001 C CNN
+F 3 "" H 9950 2950 30  0000 C CNN
+	1    9950 2950
+	0    1    1    0
+$EndComp
+$Comp
+L R R10
+U 1 1 55B4E3EA
+P 9950 3050
+F 0 "R10" V 10030 3050 50  0000 C CNN
+F 1 "1k" V 9950 3050 50  0000 C CNN
+F 2 "Resistors_SMD:R_0603" V 9880 3050 30  0001 C CNN
+F 3 "" H 9950 3050 30  0000 C CNN
+	1    9950 3050
 	0    -1   -1   0
 $EndComp
-Wire Wire Line
-	1300 8400 1300 8150
-Wire Wire Line
-	1300 8150 1350 8150
-Connection ~ 1300 8400
-Wire Wire Line
-	1950 8150 2000 8150
-Wire Wire Line
-	2000 8150 2000 8400
-Connection ~ 2000 8400
+$Comp
+L R R11
+U 1 1 55B4E3F0
+P 9950 3150
+F 0 "R11" V 10030 3150 50  0000 C CNN
+F 1 "1k" V 9950 3150 50  0000 C CNN
+F 2 "Resistors_SMD:R_0603" V 9880 3150 30  0001 C CNN
+F 3 "" H 9950 3150 30  0000 C CNN
+	1    9950 3150
+	0    1    1    0
+$EndComp
+$Comp
+L R R12
+U 1 1 55B4E3F6
+P 9950 3250
+F 0 "R12" V 10030 3250 50  0000 C CNN
+F 1 "1k" V 9950 3250 50  0000 C CNN
+F 2 "Resistors_SMD:R_0603" V 9880 3250 30  0001 C CNN
+F 3 "" H 9950 3250 30  0000 C CNN
+	1    9950 3250
+	0    -1   -1   0
+$EndComp
+Wire Wire Line
+	10100 3050 10150 3050
+Wire Wire Line
+	10100 3150 10150 3150
+Wire Wire Line
+	10100 3250 10150 3250
+Wire Wire Line
+	9700 3250 9800 3250
+Wire Wire Line
+	9800 3050 9700 3050
+Connection ~ 9700 3050
+Wire Wire Line
+	9800 3150 9700 3150
+Connection ~ 9700 3150
+$Comp
+L GND #PWR064
+U 1 1 55B512F7
+P 9700 3300
+F 0 "#PWR064" H 9700 3050 50  0001 C CNN
+F 1 "GND" H 9700 3150 50  0000 C CNN
+F 2 "" H 9700 3300 60  0000 C CNN
+F 3 "" H 9700 3300 60  0000 C CNN
+	1    9700 3300
+	1    0    0    -1
+$EndComp
+Connection ~ 9700 3250
+Wire Wire Line
+	10100 2950 10150 2950
+Wire Wire Line
+	9800 2950 9700 2950
+Wire Wire Line
+	9700 2950 9700 3300
 $EndSCHEMATC

Commit message: board modify
Parts:
- U11, U12, U13, U9: footprint Wire_Pads:SolderWirePad_single_1-5mmDrill -> user_Passive:dril_3mm
Changed lines of the file:
@@
 F 0 "U9" H 13900 9800 60  0000 C CNN
 F 1 "drill_3mm" H 13900 9150 60  0000 C CNN
-F 2 "Wire_Pads:SolderWirePad_single_1-5mmDrill" H 13900 9500 60  0001 C CNN
+F 2 "user_Passive:dril_3mm" H 13900 9500 60  0001 C CNN
 F 3 "" H 13900 9500 60  0000 C CNN
 	1    13900 9500
@@
 F 0 "U11" H 14450 9800 60  0000 C CNN
 F 1 "drill_3mm" H 14450 9150 60  0000 C CNN
-F 2 "Wire_Pads:SolderWirePad_single_1-5mmDrill" H 14450 9500 60  0001 C CNN
+F 2 "user_Passive:dril_3mm" H 14450 9500 60  0001 C CNN
 F 3 "" H 14450 9500 60  0000 C CNN
 	1    14450 9500
@@
 F 0 "U12" H 15000 9800 60  0000 C CNN
 F 1 "drill_3mm" H 15000 9150 60  0000 C CNN
-F 2 "Wire_Pads:SolderWirePad_single_1-5mmDrill" H 15000 9500 60  0001 C CNN
+F 2 "user_Passive:dril_3mm" H 15000 9500 60  0001 C CNN
 F 3 "" H 15000 9500 60  0000 C CNN
 	1    15000 9500
@@
 F 0 "U13" H 15550 9800 60  0000 C CNN
 F 1 "drill_3mm" H 15550 9150 60  0000 C CNN
-F 2 "Wire_Pads:SolderWirePad_single_1-5mmDrill" H 15550 9500 60  0001 C CNN
+F 2 "user_Passive:dril_3mm" H 15550 9500 60  0001 C CNN
 F 3 "" H 15550 9500 60  0000 C CNN
 	1    15550 9500
