File: KiCAD/HubBoard/HubBoard.sch (KiCad schematic (older format))
At the start: 64 parts, among them CN1 CONN_WHITE_5, CN2 DF22L-2P, CN3 CONN_WHITE_5, CN4 DF22R-2P, CN5 CONN_WHITE_3, CN6 CONN_WHITE_3, SW1 SLIDE_SW, U1 DF3_UART, U10 PSOC3_CY8C38_FAMILY_100, U11 drill_3mm, U12 drill_3mm, U13 drill_3mm, U2 DF3_UART, U3 DF3_UART, U4 DF3_UART, U5 TA48M05F, U6 NJM2360A, U7 Mini-B, U8 PSOC3_CY8C38_FAMILY_100, U9 drill_3mm, Y1 Crystal, Y2 Crystal

Commit message: silk add
Parts:
- added D3, D4: LED, LEDs:LED-0603, symbol LED
- added R5, R6: 1k, Resistors_SMD:R_0603, symbol R
Connections:
- wire segments 240 -> 247
- no-connect marks 102 -> 100
Other:
- moved on the sheet: R4
Changed lines of the file:
@@
 $EndDescr
-$Comp
-L PSOC3_CY8C38_FAMILY_100 U8
-U 1 1 5578950C
-P 5900 5400
-F 0 "U8" H 4300 8850 60  0000 C CNN
-F 1 "PSOC3_CY8C38_FAMILY_100" H 5900 6900 60  0000 C CNN
-F 2 "Housings_QFP:TQFP-100_14x14mm_Pitch0.5mm" H 5900 5400 60  0001 C CNN
-F 3 "" H 5900 5400 60  0000 C CNN
-	1    5900 5400
-	1    0    0    -1
-$EndComp
 $Comp
 L C-RESCUE-HubBoard C3
@@
 	1050 7450 1400 7450
 Wire Wire Line
-	1550 4500 2000 4500
+	1550 4500 2250 4500
 Wire Wire Line
 	700  5000 1800 5000
@@
 NoConn ~ 6800 1950
 NoConn ~ 6900 1950
-NoConn ~ 7000 1950
-NoConn ~ 7100 1950
 Wire Wire Line
 	5950 1950 5950 1150
@@
 L +5V #PWR060
 U 1 1 55A88E4E
-P 2000 4500
-F 0 "#PWR060" H 2000 4350 50  0001 C CNN
-F 1 "+5V" H 2000 4640 50  0000 C CNN
-F 2 "" H 2000 4500 60  0000 C CNN
-F 3 "" H 2000 4500 60  0000 C CNN
-	1    2000 4500
+P 2250 4500
+F 0 "#PWR060" H 2250 4350 50  0001 C CNN
+F 1 "+5V" H 2250 4640 50  0000 C CNN
+F 2 "" H 2250 4500 60  0000 C CNN
+F 3 "" H 2250 4500 60  0000 C CNN
+	1    2250 4500
 	1    0    0    -1
 $EndComp
@@
 L LED D2
 U 1 1 55A68D85
-P 4000 8350
-F 0 "D2" H 4000 8450 50  0000 C CNN
-F 1 "LED" H 4000 8250 50  0000 C CNN
-F 2 "LEDs:LED-3MM" H 4000 8350 60  0001 C CNN
-F 3 "" H 4000 8350 60  0000 C CNN
-	1    4000 8350
+P 2100 4700
+F 0 "D2" H 2100 4800 50  0000 C CNN
+F 1 "LED" H 2100 4600 50  0000 C CNN
+F 2 "LEDs:LED-3MM" H 2100 4700 60  0001 C CNN
+F 3 "" H 2100 4700 60  0000 C CNN
+	1    2100 4700
 	0    -1   -1   0
 $EndComp
@@
 L R R4
 U 1 1 55A68E3A
-P 4000 8700
-F 0 "R4" V 4080 8700 50  0000 C CNN
-F 1 "R" V 4000 8700 50  0000 C CNN
-F 2 "Resistors_SMD:R_0603" V 3930 8700 30  0001 C CNN
-F 3 "" H 4000 8700 30  0000 C CNN
-	1    4000 8700
+P 2100 5050
+F 0 "R4" V 2180 5050 50  0000 C CNN
+F 1 "R" V 2100 5050 50  0000 C CNN
+F 2 "Resistors_SMD:R_0603" V 2030 5050 30  0001 C CNN
+F 3 "" H 2100 5050 30  0000 C CNN
+	1    2100 5050
 	1    0    0    -1
 $EndComp
@@
 L GND #PWR061
 U 1 1 55A69589
-P 4000 8850
-F 0 "#PWR061" H 4000 8600 50  0001 C CNN
-F 1 "GND" H 4000 8700 50  0000 C CNN
-F 2 "" H 4000 8850 60  0000 C CNN
-F 3 "" H 4000 8850 60  0000 C CNN
-	1    4000 8850
-	1    0    0    -1
-$EndComp
-Connection ~ 4000 8150
+P 2100 5200
+F 0 "#PWR061" H 2100 4950 50  0001 C CNN
+F 1 "GND" H 2100 5050 50  0000 C CNN
+F 2 "" H 2100 5200 60  0000 C CNN
+F 3 "" H 2100 5200 60  0000 C CNN
+	1    2100 5200
+	1    0    0    -1
+$EndComp
 Wire Wire Line
 	12500 5950 12600 5950
@@
 	1    0    0    -1
 $EndComp
-Text GLabel 6650 1800 2    60   Input ~ 0
+Text GLabel 6650 1650 1    60   Input ~ 0
 VCCD1
 Text GLabel 6000 5750 3    60   Input ~ 0
@@
 Wire Wire Line
 	9700 2950 9700 3300
+Connection ~ 2100 4500
+$Comp
+L PSOC3_CY8C38_FAMILY_100 U8
+U 1 1 5578950C
+P 5900 5400
+F 0 "U8" H 4300 8850 60  0000 C CNN
+F 1 "PSOC3_CY8C38_FAMILY_100" H 5900 6900 60  0000 C CNN
+F 2 "Housings_QFP:TQFP-100_14x14mm_Pitch0.5mm" H 5900 5400 60  0001 C CNN
+F 3 "" H 5900 5400 60  0000 C CNN
+	1    5900 5400
+	1    0    0    -1
+$EndComp
+Wire Wire Line
+	6650 1800 6650 1650
+$Comp
+L LED D4
+U 1 1 55B7D9F9
+P 7100 1600
+F 0 "D4" H 7100 1700 50  0000 C CNN
+F 1 "LED" H 7100 1500 50  0000 C CNN
+F 2 "LEDs:LED-0603" H 7100 1600 60  0001 C CNN
+F 3 "" H 7100 1600 60  0000 C CNN
+	1    7100 1600
+	0    1    1    0
+$EndComp
+$Comp
+L LED D3
+U 1 1 55B7DABC
+P 7000 1600
+F 0 "D3" H 7000 1700 50  0000 C CNN
+F 1 "LED" H 7000 1500 50  0000 C CNN
+F 2 "LEDs:LED-0603" H 7000 1600 60  0001 C CNN
+F 3 "" H 7000 1600 60  0000 C CNN
+	1    7000 1600
+	0    1    1    0
+$EndComp
+$Comp
+L R R6
+U 1 1 55B7DB75
+P 7100 1200
+F 0 "R6" V 7180 1200 50  0000 C CNN
+F 1 "1k" V 7100 1200 50  0000 C CNN
+F 2 "Resistors_SMD:R_0603" V 7030 1200 30  0001 C CNN
+F 3 "" H 7100 1200 30  0000 C CNN
+	1    7100 1200
+	1    0    0    -1
+$EndComp
+$Comp
+L R R5
+U 1 1 55B7E3A2
+P 7000 1200
+F 0 "R5" V 7080 1200 50  0000 C CNN
+F 1 "1k" V 7000 1200 50  0000 C CNN
+F 2 "Resistors_SMD:R_0603" V 6930 1200 30  0001 C CNN
+F 3 "" H 7000 1200 30  0000 C CNN
+	1    7000 1200
+	1    0    0    -1
+$EndComp
+Wire Wire Line
+	7100 1800 7100 1950
+Wire Wire Line
+	7000 1800 7000 1950
+Wire Wire Line
+	7000 1350 7000 1400
+Wire Wire Line
+	7100 1350 7100 1400
+Wire Wire Line
+	7000 1050 7100 1050
+$Comp
+L GND #PWR065
+U 1 1 55B7F9F4
+P 7050 1000
+F 0 "#PWR065" H 7050 750 50  0001 C CNN
+F 1 "GND" H 6900 900 50  0000 C CNN
+F 2 "" H 7050 1000 60  0000 C CNN
+F 3 "" H 7050 1000 60  0000 C CNN
+	1    7050 1000
+	-1   0    0    1
+$EndComp
+Wire Wire Line
+	7050 1000 7050 1050
+Connection ~ 7050 1050
 $EndSCHEMATC
