File: KiCAD/BTM7752G/BTM7752G.sch (KiCad schematic (older format))
At the start: 27 parts, among them CN1 CONN_RED_2_Power, CN2 CONN_WHITE_5, CN3 CONN_RED_2_Power, CN4 CONN_WHITE_5_RE, CN5 CONN_RED_2_Power, P1 CONN_4_KRP, SW1 SLIDE_SW, SW2 SLIDE_SW, U1 TA48M05F, U2 BTM7752G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

Commit message: update
Parts:
- removed CN1, CN5: CONN_RED_2_Power, user_conn:CONN_RED_2P_STRAIGHT, symbol CONN_RED_2_Power
- removed SW1: SLIDE_SW, user_SW:Toggle_Swith, symbol SLIDE_SW
- added C12: 1000u, user_drill:C_Radial_D18_L36_P7.5_Horizon5, symbol CP
- added C13: 1000u, user_drill:C_Radial_D18_L36_P7.5_Horizon6, symbol CP
- added CN1: DF22L-2P, user_conn:CONN_RED_2P_STRAIGHT, symbol DF22L-2P
- added D2: LED, LEDs:LED-3MM, symbol LED
- added D3: D, user_drill:SOD-523_1, symbol D
- added R3: 10k, Resistors_SMD:R_0603, symbol R
- added R4, R5, R6: 4.7k, Resistors_SMD:R_0603, symbol R
- added U6: pad_2mm_1.7mm, user_drill:pad_2mm_1.7mm, symbol pad_2mm_1.7mm
Connections:
- net +24V: now also C12.1, C13.1, CN1.1 (Vi+), D2.2 (A), U6.1 (PIN)
- net GND: now also C12.2, C13.2, CN1.2 (Vi-), D3.2 (A), R3.2
- net IN1_1: now also R4.2; no longer U2.9 (IN1)
- net IN1_2: now also R5.2; no longer U2.10 (IN2)
- net INH1: now also R6.1; no longer U2.27 (INH)
- net IS1: now also D3.1 (K)
- new net: R5.1, U2.10 (IN2)
- new net: R6.2, U2.27 (INH)
- new net: R4.1, U2.9 (IN1)
- new net: D2.1 (K), R3.1
- no-connect marks 66 -> 63
